File: kicad/ps2_pico_hat.kicad_sch (KiCad schematic)
At the start: 17 parts, among them J1 Conn_01x20_Female_left, J3 Conn_01x20_Female_right, Q1 BSS138, Q2 BSS138, Q3 BSS138, Q4 BSS138

Commit message: Improved documentation for the hat
- Changed label on J3 to J2
- Added missing links to components
- Regenerated the iBOM with links to buy components
- Removed backup files committed in error
Parts:
- J2: renamed from J3; Amazon link (none) -> https://www.amazon.com/Female-Header-Raspberry-Expansion-Br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; Digikey link (none) -> https://www.digikey.com/en/products/detail/adafruit-industr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; Mouser link (none) -> https://www.mouser.com/ProductDetail/Samtec/RSM-120-02-S-S-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
Changed lines of the file:
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@@
   (symbol (lib_name "Conn_01x20_Female_1") (lib_id "Connector:Conn_01x20_Female") (at 62.23 168.91 180) (unit 1)
     (in_bom yes) (on_board yes)
-    (property "Reference" "J3" (id 0) (at 59.69 143.51 0)
+    (property "Reference" "J2" (id 0) (at 59.69 143.51 0)
       (effects (font (size 1.27 1.27)) (justify left))
     )
@@
     )
     (property "Datasheet" "~" (id 3) (at 62.23 168.91 0)
+      (effects (font (size 1.27 1.27)) hide)
+    )
+    (property "Mouser link" "https://www.mouser.com/ProductDetail/Samtec/RSM-120-02-S-S-TR?qs=rU5fayqh%252BE3elhTtzhxgWw%3D%3D" (id 4) (at 62.23 168.91 0)
+      (effects (font (size 1.27 1.27)) hide)
+    )
+    (property "Digikey link" "https://www.digikey.com/en/products/detail/adafruit-industries-llc/5585/16688065" (id 5) (at 62.23 168.91 0)
+      (effects (font (size 1.27 1.27)) hide)
+    )
+    (property "Amazon link" "https://www.amazon.com/Female-Header-Raspberry-Expansion-Breakout/dp/B0CFDV41T9/" (id 6) (at 62.23 168.91 0)
       (effects (font (size 1.27 1.27)) hide)
     )
@@
       (effects (font (size 1.27 1.27)) hide)
     )
-    (property "Datasheet" "https://www.mouser.com/datasheet/2/222/KMDGX-334716.pdf" (id 3) (at 170.18 203.2 0)
-      (effects (font (size 1.27 1.27)) hide)
-    )
-    (property "mouser link" "https://www.mouser.com/ProductDetail/Kycon/KMDGX-6S-BS?qs=gomZSfZNELc%252BcxHiGAVThw%3D%3D" (id 4) (at 170.18 203.2 0)
+    (property "Datasheet" "~" (id 3) (at 170.18 203.2 0)
       (effects (font (size 1.27 1.27)) hide)
     )
@@
       (effects (font (size 1.27 1.27)) hide)
     )
-    (property "Datasheet" "https://www.mouser.com/datasheet/2/222/KMDGX-334716.pdf" (id 3) (at 22.86 203.2 0)
-      (effects (font (size 1.27 1.27)) hide)
-    )
-    (property "mouser link" "https://www.mouser.com/ProductDetail/Kycon/KMDGX-6S-BS?qs=gomZSfZNELc%252BcxHiGAVThw%3D%3D" (id 4) (at 22.86 203.2 0)
+    (property "Datasheet" "~" (id 3) (at 22.86 203.2 0)
       (effects (font (size 1.27 1.27)) hide)
     )
@@
     )
     (path "/0ead8653-f9eb-4778-b668-69c178da4c0f"
-      (reference "J3") (unit 1) (value "Conn_01x20_Female_right") (footprint "Connector_PinSocket_2.54mm:PinSocket_1x20_P2.54mm_Vertical")
+      (reference "J2") (unit 1) (value "Conn_01x20_Female_right") (footprint "Connector_PinSocket_2.54mm:PinSocket_1x20_P2.54mm_Vertical")
     )
     (path "/307e5d1f-a5c8-439d-9f0d-38eabbcbad16"
